File: KiCad files/Drvce.kicad_sch (KiCad schematic)
At the start: 39 parts, among them J2 +, J3 -, SW1 SW_SPST, U1 ATtiny85-20SU

Commit message: assembly
Other:
- note added: "NEOPIXEL"
- note added: "SWITCH"
- company: (none) -> TVZ
- title: (none) -> Drvce
